File: ECAD/Eduart_IoT_Test_V_2/Eduart_Test_Platine_V2.kicad_pcb (KiCad board)
At the start: 2 copper layers, 76.8 x 54 mm, 38 parts

Commit message: Add files via upload
Other:
- board text added: "10"
- board text added: "11"
- board text added: "12"
- board text added: "A0"
- board text added: "A1"
- board text added: "A2"
- board text added: "A3"
- board text added: "A4"
- board text added: "A5"
- board text added: "D1"
- board text added: "D2"
- board text added: "D3"
- board text added: "D4"
- board text added: "D5"
- board text added: "D6"
- board text added: "D7"
- board text added: "D8"
- board text added: "D9"
Changed lines of the file:
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@@
 		(layer "Edge.Cuts")
+	)
+	(gr_text "D4"
+		(at 62.4 55.6 0)
+		(layer "Dwgs.User")
+		(effects
+			(font
+				(size 2 2)
+				(thickness 0.25)
+			)
+			(justify left bottom)
+		)
 	)
 	(gr_text "JLCJLCJLCJLC"
@@
 				(size 1 1)
 				(thickness 0.15)
+			)
+			(justify left bottom)
+		)
+	)
+	(gr_text "D1"
+		(at 50.2 55.6 0)
+		(layer "Dwgs.User")
+		(effects
+			(font
+				(size 2 2)
+				(thickness 0.25)
+			)
+			(justify left bottom)
+		)
+	)
+	(gr_text "A1"
+		(at 100.4 63.4 0)
+		(layer "Dwgs.User")
+		(effects
+			(font
+				(size 2 2)
+				(thickness 0.25)
+			)
+			(justify left bottom)
+		)
+	)
+	(gr_text "D3"
+		(at 50.2 71.6 0)
+		(layer "Dwgs.User")
+		(effects
+			(font
+				(size 2 2)
+				(thickness 0.25)
 			)
 			(justify left bottom)
@@
 		)
 	)
+	(gr_text "10"
+		(at 87.8 55.6 0)
+		(layer "Dwgs.User")
+		(effects
+			(font
+				(size 2 2)
+				(thickness 0.25)
+			)
+			(justify left bottom)
+		)
+	)
+	(gr_text "D6"
+		(at 62.4 71.6 0)
+		(layer "Dwgs.User")
+		(effects
+			(font
+				(size 2 2)
+				(thickness 0.25)
+			)
+			(justify left bottom)
+		)
+	)
+	(gr_text "A3"
+		(at 112.6 55.4 0)
+		(layer "Dwgs.User")
+		(effects
+			(font
+				(size 2 2)
+				(thickness 0.25)
+			)
+			(justify left bottom)
+		)
+	)
+	(gr_text "D7"
+		(at 75.2 55.6 0)
+		(layer "Dwgs.User")
+		(effects
+			(font
+				(size 2 2)
+				(thickness 0.25)
+			)
+			(justify left bottom)
+		)
+	)
+	(gr_text "A5"
+		(at 112.6 71.2 0)
+		(layer "Dwgs.User")
+		(effects
+			(font
+				(size 2 2)
+				(thickness 0.25)
+			)
+			(justify left bottom)
+		)
+	)
+	(gr_text "D5"
+		(at 62.4 63.6 0)
+		(layer "Dwgs.User")
+		(effects
+			(font
+				(size 2 2)
+				(thickness 0.25)
+			)
+			(justify left bottom)
+		)
+	)
+	(gr_text "A2"
+		(at 100.4 71.2 0)
+		(layer "Dwgs.User")
+		(effects
+			(font
+				(size 2 2)
+				(thickness 0.25)
+			)
+			(justify left bottom)
+		)
+	)
+	(gr_text "A0"
+		(at 100.4 55.6 0)
+		(layer "Dwgs.User")
+		(effects
+			(font
+				(size 2 2)
+				(thickness 0.25)
+			)
+			(justify left bottom)
+		)
+	)
+	(gr_text "D9"
+		(at 75.2 71.4 0)
+		(layer "Dwgs.User")
+		(effects
+			(font
+				(size 2 2)
+				(thickness 0.25)
+			)
+			(justify left bottom)
+		)
+	)
+	(gr_text "D2"
+		(at 50.2 63.6 0)
+		(layer "Dwgs.User")
+		(effects
+			(font
+				(size 2 2)
+				(thickness 0.25)
+			)
+			(justify left bottom)
+		)
+	)
+	(gr_text "A4"
+		(at 112.6 63.2 0)
+		(layer "Dwgs.User")
+		(effects
+			(font
+				(size 2 2)
+				(thickness 0.25)
+			)
+			(justify left bottom)
+		)
+	)
+	(gr_text "11"
+		(at 87.8 63.4 0)
+		(layer "Dwgs.User")
+		(effects
+			(font
+				(size 2 2)
+				(thickness 0.25)
+			)
+			(justify left bottom)
+		)
+	)
 	(gr_text "EduArt"
 		(at 97.5 79 0)
@@
 				(thickness 0.6)
 				(bold yes)
+			)
+			(justify left bottom)
+		)
+	)
+	(gr_text "12"
+		(at 87.8 71.2 0)
+		(layer "Dwgs.User")
+		(effects
+			(font
+				(size 2 2)
+				(thickness 0.25)
+			)
+			(justify left bottom)
+		)
+	)
+	(gr_text "D8"
+		(at 75.2 63.6 0)
+		(layer "Dwgs.User")
+		(effects
+			(font
+				(size 2 2)
+				(thickness 0.25)
 			)
 			(justify left bottom)
@@
 		(polygon
 			(pts
-				(xy 50 45) (xy 50 99) (xy 126 99) (xy 126 45) (xy 50 45)
-			)
-		)
+				(xy 50 45) (xy 50 99) (xy 126 99) (xy 126 45)
+			)
+		)
